File: spark/spark.kicad_sch (KiCad schematic)
At the start: 26 parts, among them J1 USB_B_Mini, Q1 SS8050-G, Q2 SS8050-G, U1 AMS1117-3.3, U2 CP2102N-Axx-xQFN28, U3 ESP32-WROOM-32

Commit message: whoops, forgot the switches
Parts:
- added C7, C8: 0.1uF/50V(10%)(NC), Capacitor_SMD:C_0402_1005Metric, symbol Device:C
- added SW1, SW2: SW_Push, symbol Switch:SW_Push
- C1: value C22uF/10V(20%) -> 22uF/10V(20%)
Connections:
- net EN: now also C8.2, SW2.2
- net GND: now also C7.1, C8.1, SW1.1, SW2.1
- net IO0: now also C7.2, SW1.2

Commit message: Working PCB #1
Parts:
- added D6: 1N4001, Diode_THT:D_DO-41_SOD81_P10.16mm_Horizontal, symbol Diode:1N4001
- added D7: RED LED, LED_SMD:LED_0805_2012Metric_Pad1.15x1.40mm_HandSolder, symbol Device:LED
- added J2: Screw_Terminal_01x03, TerminalBlock_TE-Connectivity:TerminalBlock_TE_282834-3_1x03_P2.54mm_Horizontal, symbol Connector:Screw_Terminal_01x03
- added K1: SRD-03VDC-SL-C, Relay_THT:Relay_SPDT_SANYOU_SRD_Series_Form_C_WithA, symbol Relay:Relay_SPDT
- added Q3: 2N3904, Package_TO_SOT_SMD:TSOT-23, symbol Transistor_BJT:2N3904
- added R10: 1K(5%), Resistor_SMD:R_0402_1005Metric, symbol Device:R
- added R11: 2K(5%), Resistor_SMD:R_0402_1005Metric, symbol Device:R
- SW1/BOOT1: renamed from SW1; footprint (none) -> Button_Switch_SMD:SW_Push_1P1T_NO_CK_KSC7xxJ
- SW2/EN1: renamed from SW2; footprint (none) -> Button_Switch_SMD:SW_Push_1P1T_NO_CK_KSC7xxJ
- renumbered C3 to C2, C2 to C3, C7 to C5, C8 to C6, C6 to C7, C5 to C8, D3 to D2, D4 to D3, D5 to D4, D2 to D5, R5 to R4, R4 to R5
Connections:
- net GND: now also D7.1 (K), Q3.1 (E)
- net IO18: now also R10.1, R11.2
- net VDD33: now also D6.1 (K), K1.A1
- new net: Q3.2 (B), R10.2
- new net: D6.2 (A), K1.A2, Q3.3 (C)
- new net: D7.2 (A), R11.1
- new net R1C: J2.2 (Pin_2), K1.11
- new net R1N0: J2.1 (Pin_1), K1.14
- new net R1NC: J2.3 (Pin_3), K1.12
Other:
- moved on the sheet: C5, C6, SW1/BOOT1, SW2/EN1
