File: spark/spark.kicad_pcb (KiCad board)
At the start: 2 copper layers, 2 parts, among them U1 ESP32-C6-DevKitC-1, U1 ESP32-WROOM-32D

Commit message: Working PCB #1
Parts:
- removed the U1 at (154.9, 66.0)
- removed the U1 at (54.8, 65.4)
- added C1: 22uF/10V(20%), Capacitor_SMD:C_0402_1005Metric, F.Cu at (103.8, 102.1)
- added C2: 0.1uF/50V(10%), Capacitor_SMD:C_0402_1005Metric, F.Cu at (114.6, 107.2)
- added C3: 22uF/10V(20%), Capacitor_SMD:C_0402_1005Metric, F.Cu at (107.2, 108.6)
- added C4: 4.7uF/6.3V(10%), Capacitor_SMD:C_0402_1005Metric, F.Cu at (115.4, 106.2)
- added C5: 0.1uF/50V(10%)(NC), Capacitor_SMD:C_0402_1005Metric, F.Cu at (100.1, 116.8)
- added C6: 0.1uF/50V(10%)(NC), Capacitor_SMD:C_0402_1005Metric, F.Cu at (132.8, 116.4)
- added C7: 0.1uF/50V(10%), Capacitor_SMD:C_0402_1005Metric, F.Cu at (112.4, 102.4)
- added C8: 22uF/10V(20%), Capacitor_SMD:C_0402_1005Metric, F.Cu at (112.4, 101.3)
- added D1: RED LED, LED_SMD:LED_0805_2012Metric_Pad1.15x1.40mm_HandSolder, F.Cu at (106.2, 101.0)
- added D2: ESD5Zxx, Diode_SMD:D_SOD-523, F.Cu at (113.7, 111.5)
- added D3: ESD5Zxx, Diode_SMD:D_SOD-523, F.Cu at (119.9, 111.5)
- added D4: ESD5Zxx, Diode_SMD:D_SOD-523, F.Cu at (119.9, 110.0)
- added D5: D, Diode_SMD:D_0402_1005Metric, F.Cu at (107.2, 104.5)
- added D6: 1N4001, Diode_THT:D_DO-41_SOD81_P10.16mm_Horizontal, F.Cu at (144.8, 83.4)
- added D7: RED LED, LED_SMD:LED_0805_2012Metric_Pad1.15x1.40mm_HandSolder, F.Cu at (134.6, 79.6)
- added J1: USB_B_Mini, Connector_USB:USB_Mini-B_Lumberg_2486_01_Horizontal, F.Cu at (116.3, 116.5)
- added J2: Screw_Terminal_01x03, TerminalBlock_TE-Connectivity:TerminalBlock_TE_282834-3_1x03_P2.54mm_Horizontal, F.Cu at (142.2, 113.0)
- added K1: SRD-03VDC-SL-C, Relay_THT:Relay_SPDT_SANYOU_SRD_Series_Form_C_WithA, F.Cu at (137.2, 86.8)
- added Q1: SS8050-G, Package_TO_SOT_SMD:SOT-23, F.Cu at (121.9, 96.8)
- added Q2: SS8050-G, Package_TO_SOT_SMD:SOT-23, F.Cu at (121.9, 101.3)
- added Q3: 2N3904, Package_TO_SOT_SMD:TSOT-23, F.Cu at (130.8, 82.1)
- added R1: 2K (5%), Resistor_SMD:R_0402_1005Metric, F.Cu at (105.4, 102.5)
- added R10: 1K(5%), Resistor_SMD:R_0402_1005Metric, F.Cu at (129.5, 77.5)
- added R11: 2K(5%), Resistor_SMD:R_0402_1005Metric, F.Cu at (130.8, 77.5)
- added R2: R0 (5%), Resistor_SMD:R_0402_1005Metric, F.Cu at (117.1, 96.0)
- added R3: R0 (5%), Resistor_SMD:R_0402_1005Metric, F.Cu at (116.1, 96.0)
- added R4: 10K(5%), Resistor_SMD:R_0402_1005Metric, F.Cu at (122.8, 99.1)
- added R5: 10K(5%), Resistor_SMD:R_0402_1005Metric, F.Cu at (120.9, 99.1)
- added R6: 22.1K(5%), Resistor_SMD:R_0402_1005Metric, F.Cu at (114.8, 104.4)
- added R7: 47.5K(5%), Diode_SMD:D_SOD-523, F.Cu at (113.0, 104.1)
- added R8: 2K(5%), Capacitor_SMD:C_0402_1005Metric, F.Cu at (116.0, 104.4)
- added R9: 10K(5%)(NC), Resistor_SMD:R_0402_1005Metric, F.Cu at (117.2, 104.4)
- added SW1/BOOT1: SW_Push, Button_Switch_SMD:SW_Push_1P1T_NO_CK_KSC7xxJ, F.Cu at (105.2, 116.7)
- added SW2/EN1: SW_Push, Button_Switch_SMD:SW_Push_1P1T_NO_CK_KSC7xxJ, F.Cu at (127.5, 116.4)
- added U1: AMS1117-3.3, Package_TO_SOT_SMD:SOT-223-3_TabPin2, F.Cu at (102.3, 106.7)
- added U2: CP2102N-Axx-xQFN28, Package_DFN_QFN:QFN-28-1EP_5x5mm_P0.5mm_EP3.35x3.35mm, F.Cu at (116.6, 100.2)
- added U3: ESP32-WROOM-32, RF_Module:ESP32-WROOM-32, F.Cu at (117.0, 83.2)
Routing:
- net GND: track 0.00 -> 148.0 mm, vias 0 -> 10
- net VDD33: track 0.00 -> 111.7 mm, vias 0 -> 4
- net EN: track 0.00 -> 69.0 mm, vias 0 -> 3
- net IO0: track 0.00 -> 40.9 mm
- net R1C: track 0.00 -> 26.0 mm
- net RXD0: track 0.00 -> 24.4 mm, vias 0 -> 2
- net TXD0: track 0.00 -> 23.3 mm
- net USB_DP: track 0.00 -> 22.5 mm, vias 0 -> 2
- net USB_DN: track 0.00 -> 22.3 mm, vias 0 -> 2
- net VBUS: track 0.00 -> 20.7 mm, vias 0 -> 2
- net R1N0: track 0.00 -> 17.3 mm
- net DTR: track 0.00 -> 14.5 mm, vias 0 -> 2
- net IO18: track 0.00 -> 11.5 mm
- net Net-(D6-A): track 0.00 -> 9.34 mm
- net R1NC: track 0.00 -> 7.33 mm
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- added copper zone on B.Cu, net GND
Other:
- board outline added: 53.7 x 54.2 mm

Commit message: fix all design rules issues
Parts:
- moved C6 4.96 mm to (128.3, 114.4)
- moved D2 4.96 mm to (109.1, 109.5)
- moved D3 4.96 mm to (115.3, 109.5)
- moved D4 4.96 mm to (115.3, 108.0)
- moved Q1 4.96 mm to (117.3, 94.8)
- moved R4 4.96 mm to (118.3, 97.1)
- moved R6 4.96 mm to (110.3, 102.4)
- moved SW1/BOOT1 4.96 mm to (100.6, 114.7)
- moved U1 4.96 mm to (97.7, 104.7)
- moved U3 4.96 mm to (112.4, 81.2)
- moved C1 4.96 mm to (99.2, 100.1)
- moved C2 4.96 mm to (110.0, 105.2)
- moved C8 4.96 mm to (107.9, 99.3)
- moved D1 4.96 mm to (101.6, 99.0)
- moved D5 4.96 mm to (102.6, 102.5)
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Other:
- board size 53.7 x 54.2 mm -> 49.7 x 56.8 mm

Commit message: Another checkpoint, going to do layout again for funsies
Parts:
- removed D2: ESD5Zxx, Diode_SMD:D_SOD-523
- added D2-4: ESD5Zxx, Diode_SMD:D_SOD-523, F.Cu at (99.8, 111.8)
- moved D6 46.3 mm to (112.8, 118.6), turned to 0 degrees
- moved C6 40.9 mm to (87.4, 113.3), turned to -90 degrees
- moved SW2/EN1 39.8 mm to (83.2, 117.6)
- moved Q1 35.0 mm to (85.6, 109.6), turned to -90 degrees
- moved K1 33.8 mm to (117.9, 115.2), turned to 90 degrees
- moved R4 33.2 mm to (87.9, 110.4), turned to 90 degrees
- moved R5 30.6 mm to (87.9, 108.5), turned to -90 degrees
- moved Q2 28.9 mm to (90.4, 109.6), turned to -90 degrees
- moved C8 22.9 mm to (85.0, 98.1), turned to 90 degrees
- moved J2 22.7 mm to (122.2, 94.5)
- moved C7 21.9 mm to (86.0, 98.0), turned to 90 degrees
- moved U3 20.1 mm to (93.3, 87.3), turned to 90 degrees
- moved D5 17.2 mm to (109.5, 118.3)
- moved R9 17.0 mm to (96.0, 99.1), turned to -90 degrees
- moved C1 16.2 mm to (108.7, 113.3), turned to 0 degrees
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Routing:
- net VDD33: track 111.7 -> 59.4 mm, vias 4 -> 3
- net EN: track 69.0 -> 27.4 mm, vias 3 -> 2
- net RXD: track 1.52 -> 35.2 mm, vias 0 -> 2
- net VBUS: track 20.7 -> 53.9 mm, vias 2 -> 3
- net TXD: track 1.33 -> 31.5 mm, vias 0 -> 2
- net Net-(D6-A): track 9.28 -> 35.3 mm
- net IO18: track 11.5 -> 30.4 mm, vias 0 -> 2
- net IO0: track 40.9 -> 55.7 mm, vias 0 -> 3
- net R1N0: track 17.3 -> 7.26 mm
- net RTS: track 6.18 -> 15.7 mm
- net R1NC: track 7.33 -> 15.8 mm
- net Net-(D1-A): track 2.05 -> 10.1 mm, vias 0 -> 2
- net USB_DP: track 22.5 -> 15.5 mm, vias 2 -> 0
- net GND: track 148.0 -> 141.3 mm, vias 10 -> 7
- net USB_DN: track 22.3 -> 15.8 mm
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Other:
- board size 49.7 x 56.8 mm -> 48.8 x 49.3 mm
